File: hardware/lin-pump-control/pump_control.kicad_sch (KiCad schematic)
At the start: 8 parts, among them J4 PUMP, Q3 2N7002, Q4 SUD50P04-08

Commit message: Add INA219 to pump controller, change to using regulator module
Parts:
- added R15: 100m 1% 2W, Resistor_SMD:R_2512_6332Metric_Pad1.40x3.35mm_HandSolder, symbol Device:R
- added U5: INA219BxDCN, Package_TO_SOT_SMD:SOT-23-8, symbol Beirdo:INA219BxDCN
- renumbered D4 to D3, R19 to R11, R20 to R12, R21 to R13, R22 to R14
Connections:
- net +3V3: now also U5.4 (VS)
- net GND: now also U5.3 (GND)
- net PUMP+: now also R15.1, U5.2 (IN-); no longer D3.3, Q4.2 (D), R14.1
- new net: D3.3, Q4.2 (D), R14.1, R15.2, U5.1 (IN+)
- new net SCL: U5.5 (SCL), U5.7 (A0), U5.8 (A1)
- new net SDA: U5.6 (SDA)
Other:
- note added: "I2C Address 0x40-4F (using 0x4F)"
