File: hardware/lin-coolant-temperature/thermistors.kicad_sch (KiCad schematic)
At the start: 8 parts, among them J4 10k NTC, J5 10k NTC, U6 LMV601, U7 LMV601

Commit message: Add firmware for lin-coolant-temperature, cleanup layout
Parts:
- renumbered D3 to D4, D4 to D5, R18 to R19, R19 to R20
Changed lines of the file:
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@@
   (symbol (lib_id "power:+3V3") (at 117.475 93.599 0) (unit 1)
     (in_bom yes) (on_board yes) (fields_autoplaced)
-    (property "Reference" "#PWR?" (id 0) (at 117.475 97.409 0)
+    (property "Reference" "#PWR042" (id 0) (at 117.475 97.409 0)
       (effects (font (size 1.27 1.27)) hide)
     )
@@
   (symbol (lib_id "power:GND") (at 153.924 125.476 0) (unit 1)
     (in_bom yes) (on_board yes) (fields_autoplaced)
-    (property "Reference" "#PWR?" (id 0) (at 153.924 131.826 0)
+    (property "Reference" "#PWR047" (id 0) (at 153.924 131.826 0)
       (effects (font (size 1.27 1.27)) hide)
     )
@@
   (symbol (lib_id "Device:D_Zener") (at 117.475 114.3 270) (unit 1)
     (in_bom yes) (on_board yes)
-    (property "Reference" "D3" (id 0) (at 119.634 112.395 90)
+    (property "Reference" "D4" (id 0) (at 119.634 112.395 90)
       (effects (font (size 1.27 1.27)) (justify left))
     )
@@
   (symbol (lib_id "power:GND") (at 117.475 119.38 0) (unit 1)
     (in_bom yes) (on_board yes) (fields_autoplaced)
-    (property "Reference" "#PWR?" (id 0) (at 117.475 125.73 0)
+    (property "Reference" "#PWR043" (id 0) (at 117.475 125.73 0)
       (effects (font (size 1.27 1.27)) hide)
     )
@@
   (symbol (lib_id "power:GND") (at 154.94 60.071 0) (unit 1)
     (in_bom yes) (on_board yes) (fields_autoplaced)
-    (property "Reference" "#PWR?" (id 0) (at 154.94 66.421 0)
+    (property "Reference" "#PWR049" (id 0) (at 154.94 66.421 0)
       (effects (font (size 1.27 1.27)) hide)
     )
@@
   (symbol (lib_id "power:GND") (at 118.491 53.975 0) (unit 1)
     (in_bom yes) (on_board yes) (fields_autoplaced)
-    (property "Reference" "#PWR?" (id 0) (at 118.491 60.325 0)
+    (property "Reference" "#PWR045" (id 0) (at 118.491 60.325 0)
       (effects (font (size 1.27 1.27)) hide)
     )
@@
   (symbol (lib_id "power:+3V3") (at 153.924 96.139 0) (unit 1)
     (in_bom yes) (on_board yes) (fields_autoplaced)
-    (property "Reference" "#PWR?" (id 0) (at 153.924 99.949 0)
+    (property "Reference" "#PWR046" (id 0) (at 153.924 99.949 0)
       (effects (font (size 1.27 1.27)) hide)
     )
@@
   (symbol (lib_id "Device:R") (at 117.475 99.314 0) (unit 1)
     (in_bom yes) (on_board yes) (fields_autoplaced)
-    (property "Reference" "R18" (id 0) (at 119.253 98.0439 0)
+    (property "Reference" "R19" (id 0) (at 119.253 98.0439 0)
       (effects (font (size 1.27 1.27)) (justify left))
     )
@@
   (symbol (lib_id "power:GND") (at 87.884 48.387 0) (unit 1)
     (in_bom yes) (on_board yes) (fields_autoplaced)
-    (property "Reference" "#PWR?" (id 0) (at 87.884 54.737 0)
+    (property "Reference" "#PWR041" (id 0) (at 87.884 54.737 0)
       (effects (font (size 1.27 1.27)) hide)
     )
@@
   (symbol (lib_id "Device:R") (at 118.491 33.909 0) (unit 1)
     (in_bom yes) (on_board yes) (fields_autoplaced)
-    (property "Reference" "R19" (id 0) (at 120.269 32.6389 0)
+    (property "Reference" "R20" (id 0) (at 120.269 32.6389 0)
       (effects (font (size 1.27 1.27)) (justify left))
     )
@@
   (symbol (lib_id "power:+3V3") (at 118.491 28.194 0) (unit 1)
     (in_bom yes) (on_board yes) (fields_autoplaced)
-    (property "Reference" "#PWR?" (id 0) (at 118.491 32.004 0)
+    (property "Reference" "#PWR044" (id 0) (at 118.491 32.004 0)
       (effects (font (size 1.27 1.27)) hide)
     )
@@
   (symbol (lib_id "Device:D_Zener") (at 118.491 48.895 270) (unit 1)
     (in_bom yes) (on_board yes)
-    (property "Reference" "D4" (id 0) (at 120.65 46.99 90)
+    (property "Reference" "D5" (id 0) (at 120.65 46.99 90)
       (effects (font (size 1.27 1.27)) (justify left))
     )
@@
   (symbol (lib_id "power:+3V3") (at 154.94 31.115 0) (unit 1)
     (in_bom yes) (on_board yes) (fields_autoplaced)
-    (property "Reference" "#PWR?" (id 0) (at 154.94 34.925 0)
+    (property "Reference" "#PWR048" (id 0) (at 154.94 34.925 0)
       (effects (font (size 1.27 1.27)) hide)
     )
@@
   (symbol (lib_id "power:GND") (at 86.868 113.792 0) (unit 1)
     (in_bom yes) (on_board yes) (fields_autoplaced)
-    (property "Reference" "#PWR?" (id 0) (at 86.868 120.142 0)
-      (effects (font (size 1.27 1.27)) hide)
-    )
+    (property "Reference" "#PWR040" (id 0) (at 86.868 120.142 0)
+      (effects (font (size 1.27 1.27)) hide)
+    )
