File: hardware/lin-flow-sensor/flow_meter.kicad_sch (KiCad schematic)
At the start: 6 parts, among them J4 Flow Meter, J5 Flow Meter, U6 74AHCT1G14, U7 74AHCT1G14

Commit message: Update the schematics... remove PCA9536, use voltage regulator
Parts:
- J4: value Flow Meter -> Flow 1
- J5: value Flow Meter -> Flow 2
Changed lines of the file:
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@@
   (title_block
     (title "LINBus Flow Sensor")
-    (date "2023-02-18")
+    (date "2023-03-03")
     (rev "1.0")
     (company "Gavin Hurlbut")
@@
   (symbol (lib_id "Connector:Screw_Terminal_01x03") (at 119.761 98.806 0) (mirror y) (unit 1)
     (in_bom yes) (on_board yes) (fields_autoplaced)
-    (property "Reference" "J4" (id 0) (at 119.761 90.043 0))
-    (property "Value" "Flow Meter" (id 1) (at 119.761 92.583 0))
+    (property "Reference" "J4" (id 0) (at 119.761 90.17 0))
+    (property "Value" "Flow 1" (id 1) (at 119.761 92.71 0))
     (property "Footprint" "TerminalBlock_TE-Connectivity:TerminalBlock_TE_282834-3_1x03_P2.54mm_Horizontal" (id 2) (at 119.761 98.806 0)
       (effects (font (size 1.27 1.27)) hide)
@@
     (in_bom yes) (on_board yes) (fields_autoplaced)
     (property "Reference" "J5" (id 0) (at 120.523 132.08 0))
-    (property "Value" "Flow Meter" (id 1) (at 120.523 134.62 0))
+    (property "Value" "Flow 2" (id 1) (at 120.523 134.62 0))
     (property "Footprint" "TerminalBlock_TE-Connectivity:TerminalBlock_TE_282834-3_1x03_P2.54mm_Horizontal" (id 2) (at 120.523 140.843 0)
       (effects (font (size 1.27 1.27)) hide)
