File: hardware/lin-flow-sensor/lin-flow-sensor.kicad_pcb (KiCad board)
At the start: 4 copper layers, 55.6 x 43.2 mm, 56 parts, among them J1 UPDI, J2 I2C LCD, J3 Screw_Terminal_01x03, J4 Flow 0, J5 Flow 1, Q1 2N7002, Q2 2N7002, U1 TJA1021T, U2 ATtiny824-X, U3 PCA9536DP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

Commit message: Update the schematics... remove PCA9536, use voltage regulator
Parts:
- removed C10, C11: 10uF, Capacitor_SMD:C_0805_2012Metric_Pad1.18x1.45mm_HandSolder
- removed C8: 2.2uF, Capacitor_SMD:C_0805_2012Metric_Pad1.18x1.45mm_HandSolder
- removed C9: 100uF Ta 6V, Capacitor_Tantalum_SMD:CP_EIA-3216-10_Kemet-I_Pad1.58x1.35mm_HandSolder
- removed D3: BYS10-35, Diode_SMD:D_SMA_Handsoldering
- removed JP2: A3, Jumper:SolderJumper-2_P1.3mm_Open_TrianglePad1.0x1.5mm
- removed JP3: A2, Jumper:SolderJumper-2_P1.3mm_Open_TrianglePad1.0x1.5mm
- removed JP4: A1, Jumper:SolderJumper-2_P1.3mm_Open_TrianglePad1.0x1.5mm
- removed JP5: A0, Jumper:SolderJumper-2_P1.3mm_Open_TrianglePad1.0x1.5mm
- removed L1: 33uH 5A 88mOhm, Beirdo:PM4346.333NLT
- removed R11: 357k 1%, Resistor_SMD:R_0805_2012Metric_Pad1.20x1.40mm_HandSolder
- removed R12: 100k 1%, Resistor_SMD:R_0805_2012Metric_Pad1.20x1.40mm_HandSolder
- removed R13: 909k 1%, Resistor_SMD:R_0805_2012Metric_Pad1.20x1.40mm_HandSolder
- removed R14: 324k 1%, Resistor_SMD:R_0805_2012Metric_Pad1.20x1.40mm_HandSolder
- removed R15: 47k, Resistor_SMD:R_0805_2012Metric_Pad1.20x1.40mm_HandSolder
- removed R16: 6k2, Resistor_SMD:R_0805_2012Metric_Pad1.20x1.40mm_HandSolder
- removed R17: 1k3, Resistor_SMD:R_0805_2012Metric_Pad1.20x1.40mm_HandSolder
- removed R18: 560R, Resistor_SMD:R_0805_2012Metric_Pad1.20x1.40mm_HandSolder
- removed U5: BD9G341EFJ, Package_SO:HTSOP-8-1EP_3.9x4.9mm_P1.27mm_EP2.4x3.2mm_ThermalVias
- C3: value 2.2uF -> 10uF 100V; footprint Capacitor_SMD:C_0805_2012Metric_Pad1.18x1.45mm_HandSolder -> Capacitor_SMD:C_1210_3225Metric_Pad1.33x2.70mm_HandSolder
- C4: value 10uF 100V -> 1uF; footprint Capacitor_SMD:C_1210_3225Metric_Pad1.33x2.70mm_HandSolder -> Capacitor_SMD:C_0805_2012Metric_Pad1.18x1.45mm_HandSolder
- C5: value 100nF -> 100uF Ta 6V; footprint Capacitor_SMD:C_0805_2012Metric_Pad1.18x1.45mm_HandSolder -> Capacitor_Tantalum_SMD:CP_EIA-3216-10_Kemet-I_Pad1.58x1.35mm_HandSolder
- C6: value 10nF -> 1uF
- C7: value 2.2uF -> 10uF; moved to F.Cu
- D2, JP1, R6: moved to B.Cu
- J1: footprint Beirdo:FTDI_BASIC -> Beirdo:FTDI-TARGET
- J4: value Flow 0 -> Flow 1
- J5: value Flow 1 -> Flow 2
- U3: value PCA9536DP -> Voltage Regulator; footprint Package_SO:TSSOP-8_3x3mm_P0.65mm -> Beirdo:Switching_Regulator_Module
- U4: value LTC3203BEDD-PBF -> MCP1754S-3302xCB; footprint UltraLibrarian:LTC3203BEDD-PBF -> Package_TO_SOT_SMD:SOT-23
- moved C4 33.4 mm to (181.6, 77.7), turned to 90 degrees
- moved C3 30.5 mm to (213.6, 69.5), turned to -90 degrees
- moved REF** 28.6 mm to (180.0, 68.1)
- moved C5 21.3 mm to (179.5, 77.1), turned to 90 degrees
- moved U3 15.2 mm to (187.1, 78.0), turned to 180 degrees
- moved C7 12.7 mm to (196.6, 81.2), turned to 0 degrees
- moved C6 12.0 mm to (193.2, 85.9), turned to -90 degrees
- moved U4 10.0 mm to (192.7, 81.9), turned to 90 degrees
- moved F1 3.30 mm to (215.8, 64.0), turned to 180 degrees
- moved D2 2.90 mm to (213.8, 94.9), turned to 180 degrees
- moved R6 2.12 mm to (218.4, 94.8), turned to 0 degrees
- moved JP1 0.65 mm to (222.2, 94.9)
Connections:
- C3 pad 1: +3V3 -> +12V
- C4 pad 1: +12V -> +5V
- C5 pad 1: Net-(C5-Pad1) -> +5V
- C5 pad 2: Net-(C5-Pad2) -> GND
- C6 pad 1: Net-(C6-Pad1) -> +3V3
- C6 pad 2: Net-(C6-Pad2) -> GND
- C7 pad 1: Net-(C7-Pad1) -> +5V
- C7 pad 2: Net-(C7-Pad2) -> GND
- J1 pad 1: GND -> unconnected-(J1-Pad1)
- J1 pad 2: unconnected-(J1-Pad2) -> UPDI
- J1 pad 4: Net-(J1-Pad4) -> Net-(JP1-Pad1)
- J1 pad 5: UPDI -> unconnected-(J1-Pad5)
- J1 pad 6: unconnected-(J1-Pad6) -> GND
- JP1 pad 1: Net-(J1-Pad3) -> Net-(JP1-Pad1)
- Q1 pad 1: SCL3V -> SCL
- Q1 pad 2: SCL3V -> SCL
- Q2 pad 1: SDA3V -> SDA
- Q2 pad 2: SDA3V -> SDA
- R10 pad 2: SCL3V -> SCL
- R6 pad 2: Net-(J1-Pad4) -> Net-(J1-Pad3)
- R9 pad 2: SDA3V -> SDA
- U2 pad 8: SDA3V -> SDA
- U2 pad 9: SCL3V -> SCL
- U3 pad 1: Net-(JP5-Pad2) -> +5V
- U3 pad 2: Net-(JP4-Pad2) -> GND
- U3 pad 3: Net-(JP3-Pad2) -> +12V
- U3 pad 4: GND -> unconnected-(U3-Pad4)
- U4 pad 1: Net-(C8-Pad1) -> GND
- U4 pad 2: +5V -> +3V3
- U4 pad 3: Net-(C7-Pad2) -> +5V
Routing:
- net +5V: track 81.1 -> 23.0 mm, vias 0 -> 2
- net SDA3V: track 37.3 -> 0.00 mm, vias 3 -> 0
- net SCL3V: track 32.8 -> 0.00 mm, vias 3 -> 0
- net SDA: track 0.00 -> 32.7 mm, vias 0 -> 2
- net SCL: track 0.00 -> 30.4 mm, vias 0 -> 2
- net +3V3: track 39.5 -> 22.3 mm, vias 15 -> 11
- net GND: track 37.4 -> 23.9 mm, vias 15 -> 12
- net Net-(C5-Pad2): track 13.4 -> 0.00 mm
- net Net-(JP5-Pad2): track 9.66 -> 0.00 mm, vias 2 -> 0
- net Net-(C7-Pad1): track 8.57 -> 0.00 mm, vias 2 -> 0
- net Net-(JP4-Pad2): track 8.13 -> 0.00 mm, vias 1 -> 0
- net Net-(JP3-Pad2): track 7.65 -> 0.00 mm, vias 1 -> 0
- net Net-(JP1-Pad1): track 0.00 -> 7.64 mm, vias 0 -> 1
- net UPDI: track 10.2 -> 17.8 mm, vias 0 -> 1
- net Net-(C5-Pad1): track 7.53 -> 0.00 mm, vias 2 -> 0
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- added copper zone on In1.Cu, net +5V
Other:
- board text added: "LINBus Flow Sensor"
- board text added: "v1.0"
- board text removed: "LINBus Flow Sensor v1.0"
